Commit message: fixed transmission

File: simulation_ws/src/iiwa_description/urdf/iiwa_macros.xacro (robot description, xacro)
@@ -19,5 +19,5 @@
                     <mesh filename="${meshfile}" scale="${meshscale}"/>
                 </geometry>
-                <!--<material name="light_black"/>-->
+                <material name="light_black"/>
             </visual>
         </link>
@@ -32,12 +32,13 @@
         </joint>
 	<transmission name="trans_${name}">
-	<type>transmission_interface/SimpleTransmission</type>
-	<joint name="${name}">
-		<hardwareInterface>hardware_interface/EffortJointInterface</hardwareInterface>
-	</joint>
-	<actuator name="motor_${name}">
-		<hardwareInterface>hardware_interface/EffortJointInterface</hardwareInterface>
-		<mechanicalReduction>1</mechanicalReduction>
-	</actuator>
+		<type>transmission_interface/SimpleTransmission</type>
+		<joint name="${name}">
+			<hardwareInterface>hardware_interface/EffortJointInterface</hardwareInterface>
+		</joint>
+		<actuator name="motor_${name}">
+			<hardwareInterface>hardware_interface/EffortJointInterface</hardwareInterface>
+			<mechanicalReduction>1</mechanicalReduction>
+		</actuator>
+	</transmission>
   </xacro:macro>
 </robot>

Commit message: added 7 joints controllers working

File: simulation_ws/src/iiwa_description/urdf/iiwa_macros.xacro (robot description, xacro)
@@ -19,5 +19,5 @@
                     <mesh filename="${meshfile}" scale="${meshscale}"/>
                 </geometry>
-                <material name="light_black"/>
+                <!-- <material name="light_black"/> -->
             </visual>
         </link>
