Commit message: first gazibo simulation without controllers

File: simulation_ws/src/iiwa_description/urdf/iiwa.xacro (robot description, xacro)
@@ -6,5 +6,7 @@
                     origin_xyz="0 0 0" origin_rpy="0 0 0"
                     meshfile="package://iiwa_description/meshes/link0-binary.stl"
-                    meshscale="${m_meshscale}" />
+                    meshscale="${m_meshscale}"
+                    mass="1000.0"
+                    ixx="200" ixy="0" ixz="0" iyy="200" iyz="0" izz="200"/>
     <m_joint    name="${link00_name}__${link01_name}"
                 type="revolute"
@@ -16,5 +18,7 @@
                     origin_xyz="0 0 0" origin_rpy="0 0 0"
                     meshfile="package://iiwa_description/meshes/link1-binary.stl"
-                    meshscale="${m_meshscale}" />
+                    meshscale="${m_meshscale}"
+                    mass="1000.0"
+                    ixx="200" ixy="0" ixz="0" iyy="200" iyz="0" izz="200" />
     <m_joint    name="${link01_name}__${link02_name}"
                 type="revolute"
@@ -26,5 +30,7 @@
                     origin_xyz="0 0 -0.36" origin_rpy="0 0 0"
                     meshfile="package://iiwa_description/meshes/link2-binary.stl"
-                    meshscale="${m_meshscale}" />
+                    meshscale="${m_meshscale}"
+                    mass="1000.0"
+                    ixx="200" ixy="0" ixz="0" iyy="200" iyz="0" izz="200" />
     <m_joint    name="${link02_name}__${link03_name}"
                 type="revolute"
@@ -36,5 +42,7 @@
                     origin_xyz="0 0 -0.36" origin_rpy="0 0 0"
                     meshfile="package://iiwa_description/meshes/link3-binary.stl"
-                    meshscale="${m_meshscale}" />
+                    meshscale="${m_meshscale}"
+                    mass="1000.0"
+                    ixx="200" ixy="0" ixz="0" iyy="200" iyz="0" izz="200" />
     <m_joint    name="${link03_name}__${link04_name}"
                 type="revolute"
@@ -46,5 +54,7 @@
                     origin_xyz="0 0 -0.78" origin_rpy="0 0 0"
                     meshfile="package://iiwa_description/meshes/link4-binary.stl"
-                    meshscale="${m_meshscale}" />
+                    meshscale="${m_meshscale}"
+                    mass="1000.0"
+                    ixx="200" ixy="0" ixz="0" iyy="200" iyz="0" izz="200" />
     <m_joint    name="${link04_name}__${link05_name}"
                 type="revolute"
@@ -56,5 +66,7 @@
                     origin_xyz="0 0 -0.78" origin_rpy="0 0 0"
                     meshfile="package://iiwa_description/meshes/link5-binary.stl"
-                    meshscale="${m_meshscale}" />
+                    meshscale="${m_meshscale}"
+                    mass="1000.0"
+                    ixx="200" ixy="0" ixz="0" iyy="200" iyz="0" izz="200" />
     <m_joint    name="${link05_name}__${link06_name}"
                 type="revolute"
@@ -66,5 +78,7 @@
                     origin_xyz="0 0 -1.18" origin_rpy="0 0 0"
                     meshfile="package://iiwa_description/meshes/link6-binary.stl"
-                    meshscale="${m_meshscale}" />
+                    meshscale="${m_meshscale}"
+                    mass="1000.0"
+                    ixx="200" ixy="0" ixz="0" iyy="200" iyz="0" izz="200" />
     <m_joint    name="${link06_name}__${link07_name}"
                 type="revolute"
@@ -76,5 +90,7 @@
                     origin_xyz="0 0 -1.18" origin_rpy="0 0 0"
                     meshfile="package://iiwa_description/meshes/link7-binary.stl"
-                    meshscale="${m_meshscale}" />
+                    meshscale="${m_meshscale}"
+                    mass="1000.0"
+                    ixx="200" ixy="0" ixz="0" iyy="200" iyz="0" izz="200" />
 <!--
     <link name="base_link">

File: simulation_ws/src/iiwa_description/urdf/iiwa_macros.xacro (robot description, xacro)
@@ -1,6 +1,17 @@
 <?xml version="1.0" ?>
 <robot xmlns:xacro="http://www.ros.org/wiki/xacro">
-    <xacro:macro name="m_link_mesh" params="name origin_xyz origin_rpy meshfile meshscale">
+    <xacro:macro name="m_link_mesh" params="name origin_xyz origin_rpy meshfile meshscale mass ixx ixy ixz iyy iyz izz">
         <link name="${name}">
+            <inertial>
+                <mass value="${mass}" />
+                <origin rpy="${origin_rpy}" xyz="${origin_xyz}" />
+                <inertia ixx="${ixx}" ixy="${ixy}" ixz="${ixz}" iyy="${iyy}" iyz="${iyz}" izz="${izz}" />
+            </inertial>
+            <collision>
+                <origin rpy="${origin_rpy}" xyz="${origin_xyz}" />
+                <geometry>
+                    <mesh filename="${meshfile}" scale="${meshscale}"/>
+                </geometry>
+            </collision>
             <visual>
                 <origin rpy="${origin_rpy}" xyz="${origin_xyz}" />

Commit message: added controllers

File: simulation_ws/src/iiwa_description/urdf/iiwa.xacro (robot description, xacro)
@@ -93,30 +93,7 @@
                     mass="1000.0"
                     ixx="200" ixy="0" ixz="0" iyy="200" iyz="0" izz="200" />
-<!--
-    <link name="base_link">
-        <visual>
-            <origin rpy="0 0 0" xyz="0 0 0"/>
-            <geometry>
-                <mesh filename="package://iiwa_description/meshes/link0-binary.stl" scale="0.005 0.005 0.005"/>
-            </geometry>
-        </visual>
-    </link>
-    <joint name="base_link_link_01" type="revolute">
-        <axis xyz="0 0 1"/>
-        <limit effort="1000.0" lower="-3.14" upper="3.14" velocity="0.5"/>
-        <origin rpy="0 0 0" xyz="0 0 0.5"/>
-        <parent link="base_link"/>
-        <child link="link_01"/>
-    </joint>
--->
-<!--
-    <link name="link_01">
-        <visual>
-            <origin rpy="0 0 0" xyz="0 0 0.54"/>
-            <geometry>
-                <cylinder radius="0.35" length="0.4"/>
-            </geometry>
-        </visual>
-    </link>
--->
+	<gazebo>
+		<plugin name="gazebo_ros_control" filename="libgazebo_ros_control.so">
+		</plugin>
+	</gazebo>
 </robot>

File: simulation_ws/src/iiwa_description/urdf/iiwa_macros.xacro (robot description, xacro)
@@ -31,4 +31,13 @@
             <child link="${child}" />
         </joint>
+	<transmission name="trans_${name}">
+	<type>transmission_interface/SimpleTransmission</type>
+	<joint name="${name}">
+		<hardwareInterface>hardware_interface/EffortJointInterface</hardwareInterface>
+	</joint>
+	<actuator name="motor_${name}">
+		<hardwareInterface>hardware_interface/EffortJointInterface</hardwareInterface>
+		<mechanicalReduction>1</mechanicalReduction>
+	</actuator>
   </xacro:macro>
 </robot>

Commit message: better inertial parameters for simulation

File: simulation_ws/src/iiwa_description/urdf/iiwa.xacro (robot description, xacro)
@@ -7,6 +7,6 @@
                     meshfile="package://iiwa_description/meshes/link0-binary.stl"
                     meshscale="${m_meshscale}"
-                    mass="1000.0"
-                    ixx="200" ixy="0" ixz="0" iyy="200" iyz="0" izz="200"/>
+                    mass="500"
+                    ixx="5" ixy="0" ixz="0" iyy="6" iyz="0" izz="3"/>
     <m_joint    name="${link00_name}__${link01_name}"
                 type="revolute"
@@ -14,11 +14,12 @@
                 origin_xyz="0 0 0" origin_rpy="0 0 0"
                 parent="${link00_name}" child="${link01_name}"
-                limit_e="1000.0" limit_l="-2.967" limit_u="2.967" limit_v="1.483" />
+                limit_e="${max_effort}"
+				limit_l="-2.967" limit_u="2.967" limit_v="1.483" />
     <m_link_mesh    name="${link01_name}"
                     origin_xyz="0 0 0" origin_rpy="0 0 0"
                     meshfile="package://iiwa_description/meshes/link1-binary.stl"
                     meshscale="${m_meshscale}"
-                    mass="1000.0"
-                    ixx="200" ixy="0" ixz="0" iyy="200" iyz="0" izz="200" />
+                    mass="400"
+                    ixx="10" ixy="0" ixz="0" iyy="9" iyz="0" izz="2" />
     <m_joint    name="${link01_name}__${link02_name}"
                 type="revolute"
@@ -26,11 +27,12 @@
                 origin_xyz="0 0 0.36" origin_rpy="0 0 0"
                 parent="${link01_name}" child="${link02_name}"
-                limit_e="1000.0" limit_l="-2.094" limit_u="2.094" limit_v="1.483" />
+                limit_e="${max_effort}"
+				limit_l="-2.094" limit_u="2.094" limit_v="1.483" />
     <m_link_mesh    name="${link02_name}"
                     origin_xyz="0 0 -0.36" origin_rpy="0 0 0"
                     meshfile="package://iiwa_description/meshes/link2-binary.stl"
                     meshscale="${m_meshscale}"
-                    mass="1000.0"
-                    ixx="200" ixy="0" ixz="0" iyy="200" iyz="0" izz="200" />
+                    mass="400"
+                    ixx="5" ixy="0" ixz="0" iyy="1.8" iyz="0" izz="4.4" />
     <m_joint    name="${link02_name}__${link03_name}"
                 type="revolute"
@@ -38,11 +40,12 @@
                 origin_xyz="0 0 0" origin_rpy="0 0 0"
                 parent="${link02_name}" child="${link03_name}"
-                limit_e="1000.0" limit_l="-2.967" limit_u="2.967" limit_v="1.745" />
+                limit_e="${max_effort}"
+				limit_l="-2.967" limit_u="2.967" limit_v="1.745" />
     <m_link_mesh    name="${link03_name}"
                     origin_xyz="0 0 -0.36" origin_rpy="0 0 0"
                     meshfile="package://iiwa_description/meshes/link3-binary.stl"
                     meshscale="${m_meshscale}"
-                    mass="1000.0"
-                    ixx="200" ixy="0" ixz="0" iyy="200" iyz="0" izz="200" />
+                    mass="300"
+                    ixx="8" ixy="0" ixz="0" iyy="7.5" iyz="0" izz="1" />
     <m_joint    name="${link03_name}__${link04_name}"
                 type="revolute"
@@ -50,11 +53,12 @@
                 origin_xyz="0 0 0.42" origin_rpy="0 0 0"
                 parent="${link03_name}" child="${link04_name}"
-                limit_e="1000.0" limit_l="-2.094" limit_u="2.094" limit_v="1.309" />
+                limit_e="${max_effort}"
+				limit_l="-2.094" limit_u="2.094" limit_v="1.309" />
     <m_link_mesh    name="${link04_name}"
                     origin_xyz="0 0 -0.78" origin_rpy="0 0 0"
                     meshfile="package://iiwa_description/meshes/link4-binary.stl"
                     meshscale="${m_meshscale}"
-                    mass="1000.0"
-                    ixx="200" ixy="0" ixz="0" iyy="200" iyz="0" izz="200" />
+                    mass="270"
+                    ixx="3" ixy="0" ixz="0" iyy="1" iyz="0" izz="2.9" />
     <m_joint    name="${link04_name}__${link05_name}"
                 type="revolute"
@@ -62,11 +66,12 @@
                 origin_xyz="0 0 0" origin_rpy="0 0 0"
                 parent="${link04_name}" child="${link05_name}"
-                limit_e="1000.0" limit_l="-2.967" limit_u="2.967" limit_v="2.269" />
+                limit_e="${max_effort}"
+				limit_l="-2.967" limit_u="2.967" limit_v="2.269" />
     <m_link_mesh    name="${link05_name}"
                     origin_xyz="0 0 -0.78" origin_rpy="0 0 0"
                     meshfile="package://iiwa_description/meshes/link5-binary.stl"
                     meshscale="${m_meshscale}"
-                    mass="1000.0"
-                    ixx="200" ixy="0" ixz="0" iyy="200" iyz="0" izz="200" />
+                    mass="170"
+                    ixx="2" ixy="0" ixz="0" iyy="1.8" iyz="0" izz="0.5" />
     <m_joint    name="${link05_name}__${link06_name}"
                 type="revolute"
@@ -74,11 +79,12 @@
                 origin_xyz="0 0 0.4" origin_rpy="0 0 0"
                 parent="${link05_name}" child="${link06_name}"
-                limit_e="1000.0" limit_l="-2.094" limit_u="2.094" limit_v="2.356" />
+                limit_e="${max_effort}"
+				limit_l="-2.094" limit_u="2.094" limit_v="2.356" />
     <m_link_mesh    name="${link06_name}"
                     origin_xyz="0 0 -1.18" origin_rpy="0 0 0"
                     meshfile="package://iiwa_description/meshes/link6-binary.stl"
                     meshscale="${m_meshscale}"
-                    mass="1000.0"
-                    ixx="200" ixy="0" ixz="0" iyy="200" iyz="0" izz="200" />
+                    mass="150"
+                    ixx="0.5" ixy="0" ixz="0" iyy="0.36" iyz="0" izz="0.47" />
     <m_joint    name="${link06_name}__${link07_name}"
                 type="revolute"
@@ -86,11 +92,12 @@
                 origin_xyz="0 0 0" origin_rpy="0 0 0"
                 parent="${link06_name}" child="${link07_name}"
-                limit_e="1000.0" limit_l="-3.054" limit_u="3.054" limit_v="2.356" />
+                limit_e="${max_effort}"
+				limit_l="-3.054" limit_u="3.054" limit_v="2.356" />
     <m_link_mesh    name="${link07_name}"
                     origin_xyz="0 0 -1.18" origin_rpy="0 0 0"
                     meshfile="package://iiwa_description/meshes/link7-binary.stl"
                     meshscale="${m_meshscale}"
-                    mass="1000.0"
-                    ixx="200" ixy="0" ixz="0" iyy="200" iyz="0" izz="200" />
+                    mass="30"
+                    ixx="0.1" ixy="0" ixz="0" iyy="0.1" iyz="0" izz="0.1" />
 	<gazebo>
 		<plugin name="gazebo_ros_control" filename="libgazebo_ros_control.so">

File: simulation_ws/src/iiwa_description/urdf/iiwa_parameters.xacro (robot description, xacro)
@@ -10,3 +10,4 @@
     <xacro:property name="link07_name" value="link_07" />
     <xacro:property name="m_meshscale" value="0.001 0.001 0.001" />
+	<xacro:property name="max_effort" value="1000" />
 </robot>
